Commit message: update spider

File: src/spider_simple.urdf (robot description, URDF)
Before this commit: robot pi_robot, 13 links, 12 joints
Links:
- link base_link: geometry collision box size=0.125 0.125 0.035; visual box size=0.125 0.125 0.035
Joints:
- joint left_back_joint: origin xyz=-0.045 0.06 0 rpy=0 0 0 -> xyz=-0.045 0.045 0 rpy=0 0 0
- joint left_front_joint: origin xyz=0.045 0.06 0 rpy=0 0 0 -> xyz=0.045 0.045 0 rpy=0 0 0
- joint right_back_joint: origin xyz=-0.045 -0.06 0 rpy=0 0 0 -> xyz=-0.045 -0.045 0 rpy=0 0 0
- joint right_front_joint: origin xyz=0.045 -0.06 0 rpy=0 0 0 -> xyz=0.045 -0.045 0 rpy=0 0 0
